File: kicad/shiny-time.kicad_sch (KiCad schematic)
At the start: 44 parts, among them J1 Adafruit USB-C Power-Only Jac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, J2 Raspberry Pi Zero 2W, J3 QWIIC Connector, J4 JST-XH Buttons, J5 JST-XH Setup Button, J6 JST-XH Spare, J7 Conn_01x03_Pin, Q1 BS170, Q2 BS170, Q3 2N7000, U1 LD1117V33, U2 MCP23017x-x-SP, U3 TCA9517D, U4 DS1307+, Y1 32.768kHz

Commit message: ERC fixes
Connections:
- net BUZZ_FILTERED: now also Q3.3 (D)
- net GND: now also J1.SH (SHIELD), Q3.2 (G)
- net at BZ1.2 (-), D2.2 (A): now also Q3.1 (S)
- no-connect marks 5 -> 34
Other:
- moved on the sheet: Q3

Commit message: Assign footprints and start pcb
Parts:
- C1: footprint (none) -> Capacitor_THT:CP_Radial_D5.0mm_P2.00mm; Digikey_PN (none) -> 1189-1224-ND
- C2: footprint (none) -> Capacitor_THT:CP_Radial_D5.0mm_P2.00mm; Digikey_PN (none) -> 1189-1148-ND
- C3, C4, C5, C6, C7: footprint (none) -> Capacitor_THT:C_Disc_D5.0mm_W2.5mm_P2.50mm; Digikey_PN (none) -> 399-4264-ND
- C8: Digikey_PN (none) -> 399-18542-ND
- C9: footprint (none) -> Capacitor_THT:C_Disc_D5.0mm_W2.5mm_P5.00mm; Digikey_PN (none) -> 399-13968-ND
- D1: Digikey_PN (none) -> 497-2495-1-ND
- D2: Digikey_PN (none) -> 1N4148FS-ND
- J2: footprint Connector_PinHeader_2.54mm:PinHeader_2x20_P2.54mm_Vertical -> Connector_PinSocket_2.54mm:PinSocket_2x20_P2.54mm_Vertical; Digikey_PN (none) -> 2223-SSK04-FPH-254-B20-ND
- Q1, Q2: footprint Package_TO_SOT_THT:TO-92_HandSolder -> Package_TO_SOT_THT:TO-92_Inline; Digikey_PN (none) -> BS170-ND
- Q3: Digikey_PN (none) -> 2N7000FS-ND
- R1, R15, R2, R3, R4, R5, R6: footprint (none) -> Resistor_THT:R_Axial_DIN0204_L3.6mm_D1.6mm_P5.08mm_Horizontal; Digikey_PN (none) -> CF18JT10K0CT-ND
- R10, R12, R13, R7, R8, R9: footprint (none) -> Resistor_THT:R_Axial_DIN0204_L3.6mm_D1.6mm_P5.08mm_Horizontal; Digikey_PN (none) -> CF18JT220RCT-ND
- R11: footprint (none) -> Resistor_THT:R_Axial_DIN0204_L3.6mm_D1.6mm_P5.08mm_Horizontal; Digikey_PN (none) -> CF18JT1K00CT-ND
- R14: footprint (none) -> Resistor_THT:R_Axial_DIN0204_L3.6mm_D1.6mm_P5.08mm_Horizontal; Digikey_PN (none) -> CF18JT100RCT-ND
- R16, R17: footprint (none) -> Resistor_THT:R_Axial_DIN0204_L3.6mm_D1.6mm_P5.08mm_Horizontal; Digikey_PN (none) -> S5.1KCACT-ND
- U1: Digikey_PN (none) -> 497-1491-5-ND
- U2: Digikey_PN (none) -> MCP23017-E/SP-ND
- U3: Digikey_PN (none) -> 296-39221-1-ND
- U4: Digikey_PN (none) -> DS1307+-ND
- Y1: footprint (none) -> Crystal:Crystal_Round_D2.0mm_Vertical; Digikey_PN (none) -> 535-9032-ND

Commit message: More schematic work
Parts:
- J2: footprint Connector_PinSocket_2.54mm:PinSocket_2x20_P2.54mm_Vertical -> Module:Raspberry_Pi_Zero_Socketed_THT_FaceDown_MountingHoles
- J7: value Conn_01x03_Pin -> SPDT; footprint Connector_PinHeader_2.54mm:PinHeader_1x03_P2.54mm_Vertical -> Button_Switch_THT:SW_E-Switch_EG1271_SPDT; symbol Connector:Conn_01x03_Pin -> Switch:SW_SPDT; Digikey_PN (none) -> EG1918-ND
Connections:
- net +3.3V: now also J7.1 (A); no longer J7.3 (Pin_3)
- net +5V: now also J7.3 (C); no longer J7.1 (Pin_1)
Changed lines of the file:
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@@
 	(wire
 		(pts
+			(xy 35.56 138.43) (xy 35.56 129.54)
+		)
+		(stroke
+			(width 0)
+			(type default)
+		)
+	)
+	(wire
+		(pts
 			(xy 46.99 100.33) (xy 33.02 100.33)
 		)
@@
 	(wire
 		(pts
-			(xy 30.48 137.16) (xy 30.48 139.7)
-		)
-		(stroke
-			(width 0)
-			(type default)
-		)
-	)
-	(wire
-		(pts
 			(xy 220.98 30.48) (xy 204.47 30.48)
 		)
@@
 	(wire
 		(pts
+			(xy 54.61 130.81) (xy 50.8 130.81)
+		)
+		(stroke
+			(width 0)
+			(type default)
+		)
+	)
+	(wire
+		(pts
 			(xy 219.71 135.89) (xy 223.52 135.89)
 		)
@@
 	(wire
 		(pts
-			(xy 54.61 137.16) (xy 54.61 139.7)
-		)
-		(stroke
-			(width 0)
-			(type default)
-		)
-	)
-	(wire
-		(pts
 			(xy 43.18 142.24) (xy 53.34 142.24)
 		)
@@
 	(wire
 		(pts
-			(xy 134.62 17.78) (xy 144.78 17.78)
+			(xy 35.56 129.54) (xy 40.64 129.54)
 		)
 		(stroke
@@
 	(wire
 		(pts
-			(xy 54.61 139.7) (xy 45.72 139.7)
+			(xy 134.62 17.78) (xy 144.78 17.78)
 		)
 		(stroke
@@
 	(wire
 		(pts
+			(xy 50.8 130.81) (xy 50.8 127)
+		)
+		(stroke
+			(width 0)
+			(type default)
+		)
+	)
+	(wire
+		(pts
 			(xy 17.78 80.01) (xy 46.99 80.01)
 		)
@@
 	(wire
 		(pts
+			(xy 30.48 138.43) (xy 30.48 137.16)
+		)
+		(stroke
+			(width 0)
+			(type default)
+		)
+	)
+	(wire
+		(pts
 			(xy 46.99 39.37) (xy 58.42 39.37)
 		)
@@
 	(wire
 		(pts
-			(xy 30.48 139.7) (xy 40.64 139.7)
+			(xy 33.02 157.48) (xy 33.02 158.75)
 		)
 		(stroke
@@
 	(wire
 		(pts
-			(xy 33.02 157.48) (xy 33.02 158.75)
+			(xy 99.06 88.9) (xy 114.3 88.9)
 		)
 		(stroke
@@
 	(wire
 		(pts
-			(xy 99.06 88.9) (xy 114.3 88.9)
+			(xy 45.72 127) (xy 45.72 129.54)
+		)
+		(stroke
+			(width 0)
+			(type default)
+		)
+	)
+	(wire
+		(pts
+			(xy 50.8 127) (xy 45.72 127)
 		)
 		(stroke
@@
 	(wire
 		(pts
+			(xy 30.48 138.43) (xy 35.56 138.43)
+		)
+		(stroke
+			(width 0)
+			(type default)
+		)
+	)
+	(wire
+		(pts
 			(xy 121.92 162.56) (xy 125.73 162.56)
 		)
@@
 			)
 		)
-		(property "Footprint" "Connector_PinSocket_2.54mm:PinSocket_2x20_P2.54mm_Vertical"
+		(property "Footprint" "Module:Raspberry_Pi_Zero_Socketed_THT_FaceDown_MountingHoles"
 			(at 226.06 48.26 0)
 			(hide yes)
@@
 	)
 	(symbol
-		(lib_id "Connector:Conn_01x03_Pin")
-		(at 43.18 134.62 270)
+		(lib_id "Switch:SW_SPDT")
+		(at 43.18 134.62 90)
 		(unit 1)
 		(body_style 1)
@@
 		(fields_autoplaced yes)
 		(property "Reference" "J7"
-			(at 43.18 129.54 90)
+			(at 48.26 133.3499 90)
 			(show_name no)
 			(do_not_autoplace no)
@@
 					(size 1.27 1.27)
 				)
+				(justify right)
 			)
 		)
-		(property "Value" "Conn_01x03_Pin"
-			(at 43.18 132.08 90)
+		(property "Value" "SPDT"
+			(at 48.26 135.8899 90)
 			(show_name no)
 			(do_not_autoplace no)
@@
 					(size 1.27 1.27)
 				)
+				(justify right)
 			)
 		)
-		(property "Footprint" "Connector_PinHeader_2.54mm:PinHeader_1x03_P2.54mm_Vertical"
+		(property "Footprint" "Button_Switch_THT:SW_E-Switch_EG1271_SPDT"
 			(at 43.18 134.62 0)
 			(hide yes)
@@
 		)
 		(property "Datasheet" ""
-			(at 43.18 134.62 0)
+			(at 50.8 134.62 0)
 			(hide yes)
 			(show_name no)
@@
 			)
 		)
-		(property "Description" "Generic connector, single row, 01x03, script generated"
+		(property "Description" "Switch, single pole double throw"
 			(at 43.18 134.62 0)
 			(hide yes)
@@
 			)
 		)
-		(property "Digikey_PN" ""
+		(property "Digikey_PN" "EG1918-ND"
 			(at 43.18 134.62 90)
 			(hide yes)
@@
 	(symbol
 		(lib_id "power:+5V")
-		(at 54.61 137.16 0)
+		(at 54.61 130.81 0)
 		(unit 1)
 		(body_style 1)
@@
 		(fields_autoplaced yes)
 		(property "Reference" "#PWR024"
-			(at 54.61 140.97 0)
+			(at 54.61 134.62 0)
 			(hide yes)
 			(show_name no)
@@
 		)
 		(property "Value" "+5V"
-			(at 54.61 132.08 0)
+			(at 54.61 125.73 0)
 			(show_name no)
 			(do_not_autoplace no)
@@
 		)
 		(property "Footprint" ""
-			(at 54.61 137.16 0)
+			(at 54.61 130.81 0)
 			(hide yes)
 			(show_name no)
@@
 		)
 		(property "Datasheet" ""
-			(at 54.61 137.16 0)
+			(at 54.61 130.81 0)
 			(hide yes)
 			(show_name no)
@@
 		)
 		(property "Description" "Power symbol creates a global label with name \"+5V\""
-			(at 54.61 137.16 0)
+			(at 54.61 130.81 0)
 			(hide yes)
 			(show_name no)
